Commit message: runtime: add robot runtime contract and so101 runtime unit
Introduce robot_runtime (capability vocabulary, facade, mock, conformance,
public interface description with model metadata) and ibrobot_msgs runtime
and motion services. Add feetech_sdk and so101 sdk/hardware/description/
motion/suite packages under src/robots/, relocate so101_hardware, add the
two-direction independence gate with a fixed runtime allow-list.

- Harden SO101SystemHardware bus access with bounded retries and
  consecutive-failure counting; fail the controller chain only after
  sustained read or write failures with the Feetech fault code logged.
- Spawn the read-only leader input source from the runtime profile
  (teleoperation.leader_source) with scattered declared parameters;
  serial and calibration stay runtime-owned.
- Derive public gripper limits from calibration authority on physical
  hardware and model the arm joints with the single-turn mechanical
  envelope.
- Point the OpenHarmony cross-build and release path lists, ruff
  first-party names, the core-gate exclusion list and the repository
  layout docs at src/robots/so101 and robot_runtime.

- Harden the runtime stop path: epoch fencing keeps a concurrent mode
  switch from reviving motion or clearing a fresh stop latch, cancel
  results are validated for the active mode's trajectory endpoints, and
  stop success requires the command controllers to be deactivated.
- Harden the Feetech bus: shared config validation before EPROM writes,
  registry updates on reconfiguration, duplicate/oversized sync-read
  rejection, subset-sized sync-read sessions, sign-magnitude speed
  clamping, rollback outcome surfacing, EAGAIN-safe serial writes,
  wheel-mode calibration skip, ping-based activation diagnostics, and a
  time-budgeted retry window derived from update_rate.
- Make the core independence gate honest: launch output goes to a log
  file, motion waits are bounded, and StopRuntime(HOLD) is actually
  called with latch, lifecycle and mode asserted; pin the LeKiwi
  FTServo fetch to the feetech_sdk revision.
- Fail closed before the first runtime status in the motion server with
  a parameterized freshness deadline; honor ROS_HOME and the calibrator
  key set when loading ISP overrides.

Co-Authored-By: gpt-6-astra
Co-Authored-By: glm-5.3
Co-Authored-By: claude-opus-5
Signed-off-by: XiaoqiangWu <wuxiaoqiang.rtos@huawei.com>

File: src/robot_description/urdf/lerobot/so101/so101.urdf.xacro (robot description, xacro)
@@ -1,8 +1,6 @@
 <?xml version="1.0"?>
 <robot xmlns:xacro="http://www.ros.org/wiki/xacro" name="so101">
-    <xacro:arg name="use_sim" default="true"/>
-    <xacro:include filename="$(find robot_description)/urdf/lerobot/so101/so101_base.xacro" />
-    <xacro:include filename="$(find robot_description)/urdf/lerobot/so101/so101_gazebo.xacro" />
-    <xacro:include filename="$(find robot_description)/urdf/lerobot/so101/so101_ros2_control.xacro" />
-    <!-- cameras are generated dynamically from YAML peripherals by control.py -->
+	<!-- SSOT wrapper: the model lives in so101_description; this copy only
+	     redirects legacy consumers so the two trees can never diverge. -->
+	<xacro:include filename="$(find so101_description)/urdf/lerobot/so101/so101.urdf.xacro" />
 </robot>

File: src/robot_description/urdf/lerobot/so101/so101_base.xacro (robot description, xacro)
@@ -1,487 +1,5 @@
 <?xml version="1.0"?>
-<!--
-  This file is based on the SO-ARM100 model from:
-  https://github.com/TheRobotStudio/SO-ARM100
-  and has been modified accordingly.
--->
 <robot xmlns:xacro="http://www.ros.org/wiki/xacro">
-	<!--
-	  TCP (Tool Center Point) offset along the gripper finger extension.
-	  The SO-101 fingers extend along the gripper link's -Z axis (the jaw tip
-	  delta from the gripper origin is dominantly -Z), so a point on this line
-	  sits out at the jaws. Default 0.09 m places the TCP between the two jaw
-	  faces (single source of truth for the TCP geometry).
-	  A small -X offset re-centers the TCP onto the jaw mid-line.
-	-->
-	<xacro:arg name="tcp_offset_x" default="-0.005" />
-	<xacro:arg name="tcp_offset_z" default="-0.095" />
-	<!-- Links -->
-	<link name="world" />
-	<joint name="base_joint" type="fixed">
-		<parent link="world" />
-		<child link="base" />
-		<origin xyz="0 0 0" rpy="0 0 0" />
-	</joint>
-	<!-- Materials -->
-	<material name="3d_printed">
-		<color rgba="1.0 0.82 0.12 1.0" />
-	</material>
-	<material name="sts3215">
-		<color rgba="0.1 0.1 0.1 1.0" />
-	</material>
-	<!-- Link base -->
-	<link name="base">
-		<inertial>
-			<origin xyz="0.020739 0.00204287 0.065966" rpy="0 0 0" />
-			<mass value="0.147" />
-			<inertia ixx="0.000136117" ixy="4.59787e-07" ixz="9.75275e-08" iyy="0.000114686"
-				iyz="-4.97151e-06" izz="0.000130364" />
-		</inertial>
-		<!-- Part base_motor_holder_so101_v1 -->
-		<visual>
-			<origin xyz="0.0206915 0.0221255 0.0300817" rpy="1.5708 -1.23909e-16 2.33147e-15" />
-			<geometry>
-				<mesh
-					filename="package://robot_description/meshes/lerobot/so101/base_motor_holder_so101_v1.stl" />
-			</geometry>
-			<material name="3d_printed" />
-		</visual>
-		<collision>
-			<origin xyz="0.0206915 0.0221255 0.0300817" rpy="1.5708 -1.23909e-16 2.33147e-15" />
-			<geometry>
-				<mesh
-					filename="package://robot_description/meshes/lerobot/so101/base_motor_holder_so101_v1.stl" />
-			</geometry>
-		</collision>
-		<!-- Part base_so101_v2 -->
-		<visual>
-			<origin xyz="0.0207909 0.0221255 0.0300817" rpy="1.5708 -0 0" />
-			<geometry>
-				<mesh filename="package://robot_description/meshes/lerobot/so101/base_so101_v2.stl" />
-			</geometry>
-			<material name="3d_printed" />
-		</visual>
-		<collision>
-			<origin xyz="0.0207909 0.0221255 0.0300817" rpy="1.5708 -0 0" />
-			<geometry>
-				<mesh filename="package://robot_description/meshes/lerobot/so101/base_so101_v2.stl" />
-			</geometry>
-		</collision>
-		<!-- Part sts3215_03a_v1 -->
-		<visual>
-			<origin xyz="0.0207909 -0.0105745 0.0761817" rpy="-2.20282e-15 2.77556e-17 -1.5708" />
-			<geometry>
-				<mesh filename="package://robot_description/meshes/lerobot/so101/sts3215_03a_v1.stl" />
-			</geometry>
-			<material name="sts3215" />
-		</visual>
-		<collision>
-			<origin xyz="0.0207909 -0.0105745 0.0761817" rpy="-2.20282e-15 2.77556e-17 -1.5708" />
-			<geometry>
-				<mesh filename="package://robot_description/meshes/lerobot/so101/sts3215_03a_v1.stl" />
-			</geometry>
-		</collision>
-		<!-- Part waveshare_mounting_plate_so101_v2 -->
-		<visual>
-			<origin xyz="0.0205915 0.0467435 0.0798817" rpy="1.5708 -1.21716e-14 2.33147e-15" />
-			<geometry>
-				<mesh
-					filename="package://robot_description/meshes/lerobot/so101/waveshare_mounting_plate_so101_v2.stl" />
-			</geometry>
-			<material name="3d_printed" />
-		</visual>
-		<collision>
-			<origin xyz="0.0205915 0.0467435 0.0798817" rpy="1.5708 -1.21716e-14 2.33147e-15" />
-			<geometry>
-				<mesh
-					filename="package://robot_description/meshes/lerobot/so101/waveshare_mounting_plate_so101_v2.stl" />
-			</geometry>
-		</collision>
-	</link>
-	<!-- Link shoulder -->
-	<link name="shoulder">
-		<inertial>
-			<origin xyz="-0.0307604 -1.66727e-05 -0.0252713" rpy="0 0 0" />
-			<mass value="0.100006" />
-			<inertia ixx="8.3759e-05" ixy="7.55525e-08" ixz="-1.16342e-06" iyy="8.10403e-05"
-				iyz="1.54663e-07" izz="2.39783e-05" />
-		</inertial>
-		<!-- Part sts3215_03a_v1_2 -->
-		<visual>
-			<origin xyz="-0.0303992 0.000422241 -0.0417" rpy="1.5708 1.5708 0" />
-			<geometry>
-				<mesh filename="package://robot_description/meshes/lerobot/so101/sts3215_03a_v1.stl" />
-			</geometry>
-			<material name="sts3215" />
-		</visual>
-		<collision>
-			<origin xyz="-0.0303992 0.000422241 -0.0417" rpy="1.5708 1.5708 0" />
-			<geometry>
-				<mesh filename="package://robot_description/meshes/lerobot/so101/sts3215_03a_v1.stl" />
-			</geometry>
-		</collision>
-		<!-- Part motor_holder_so101_base_v1 -->
-		<visual>
-			<origin xyz="-0.0675992 -0.000177759 0.0158499" rpy="1.5708 -1.5708 0" />
-			<geometry>
-				<mesh
-					filename="package://robot_description/meshes/lerobot/so101/motor_holder_so101_base_v1.stl" />
-			</geometry>
-			<material name="3d_printed" />
-		</visual>
-		<collision>
-			<origin xyz="-0.0675992 -0.000177759 0.0158499" rpy="1.5708 -1.5708 0" />
-			<geometry>
-				<mesh
-					filename="package://robot_description/meshes/lerobot/so101/motor_holder_so101_base_v1.stl" />
-			</geometry>
-		</collision>
-		<!-- Part rotation_pitch_so101_v1 -->
-		<visual>
-			<origin xyz="0.0122008 2.22413e-05 0.0464" rpy="-1.5708 -0 0" />
-			<geometry>
-				<mesh
-					filename="package://robot_description/meshes/lerobot/so101/rotation_pitch_so101_v1.stl" />
-			</geometry>
-			<material name="3d_printed" />
-		</visual>
-		<collision>
-			<origin xyz="0.0122008 2.22413e-05 0.0464" rpy="-1.5708 -0 0" />
-			<geometry>
-				<mesh
-					filename="package://robot_description/meshes/lerobot/so101/rotation_pitch_so101_v1.stl" />
-			</geometry>
-		</collision>
-	</link>
-	<!-- Link upper_arm -->
-	<link name="upper_arm">
-		<inertial>
-			<origin xyz="-0.0898471 -0.00838224 0.0184089" rpy="0 0 0" />
-			<mass value="0.103" />
-			<inertia ixx="4.08002e-05" ixy="-1.97819e-05" ixz="-4.03016e-08" iyy="0.000147318"
-				iyz="8.97326e-09" izz="0.000142487" />
-		</inertial>
-		<!-- Part sts3215_03a_v1_3 -->
-		<visual>
-			<origin xyz="-0.11257 -0.0155 0.0187" rpy="-3.14159 -6.8695e-16 -1.5708" />
-			<geometry>
-				<mesh filename="package://robot_description/meshes/lerobot/so101/sts3215_03a_v1.stl" />
-			</geometry>
-			<material name="sts3215" />
-		</visual>
-		<collision>
-			<origin xyz="-0.11257 -0.0155 0.0187" rpy="-3.14159 -6.8695e-16 -1.5708" />
-			<geometry>
-				<mesh filename="package://robot_description/meshes/lerobot/so101/sts3215_03a_v1.stl" />
-			</geometry>
-		</collision>
-		<!-- Part upper_arm_so101_v1 -->
-		<visual>
-			<origin xyz="-0.065085 0.012 0.0182" rpy="3.14159 -9.35612e-32 0" />
-			<geometry>
-				<mesh filename="package://robot_description/meshes/lerobot/so101/upper_arm_so101_v1.stl" />
-			</geometry>
-			<material name="3d_printed" />
-		</visual>
-		<collision>
-			<origin xyz="-0.065085 0.012 0.0182" rpy="3.14159 -9.35612e-32 0" />
-			<geometry>
-				<mesh filename="package://robot_description/meshes/lerobot/so101/upper_arm_so101_v1.stl" />
-			</geometry>
-		</collision>
-	</link>
-	<!-- Link lower_arm -->
-	<link name="lower_arm">
-		<inertial>
-			<origin xyz="-0.0980701 0.00324376 0.0182831" rpy="0 0 0" />
-			<mass value="0.104" />
-			<inertia ixx="2.87438e-05" ixy="7.41152e-06" ixz="1.26409e-06" iyy="0.000159844"
-				iyz="-4.90188e-08" izz="0.00014529" />
-		</inertial>
-		<!-- Part under_arm_so101_v1 -->
-		<visual>
-			<origin xyz="-0.0648499 -0.032 0.0182" rpy="-3.14159 -0 3.9443e-31" />
-			<geometry>
-				<mesh filename="package://robot_description/meshes/lerobot/so101/under_arm_so101_v1.stl" />
-			</geometry>
-			<material name="3d_printed" />
-		</visual>
-		<collision>
-			<origin xyz="-0.0648499 -0.032 0.0182" rpy="-3.14159 -0 3.9443e-31" />
-			<geometry>
-				<mesh filename="package://robot_description/meshes/lerobot/so101/under_arm_so101_v1.stl" />
-			</geometry>
-		</collision>
-		<!-- Part motor_holder_so101_wrist_v1 -->
-		<visual>
-			<origin xyz="-0.0648499 -0.032 0.018" rpy="-3.14159 4.73317e-30 7.88861e-31" />
-			<geometry>
-				<mesh
-					filename="package://robot_description/meshes/lerobot/so101/motor_holder_so101_wrist_v1.stl" />
-			</geometry>
-			<material name="3d_printed" />
-		</visual>
-		<collision>
-			<origin xyz="-0.0648499 -0.032 0.018" rpy="-3.14159 4.73317e-30 7.88861e-31" />
-			<geometry>
-				<mesh
-					filename="package://robot_description/meshes/lerobot/so101/motor_holder_so101_wrist_v1.stl" />
-			</geometry>
-		</collision>
-		<!-- Part sts3215_03a_v1_4 -->
-		<visual>
-			<origin xyz="-0.1224 0.0052 0.0187" rpy="-3.14159 -3.58047e-15 -3.14159" />
-			<geometry>
-				<mesh filename="package://robot_description/meshes/lerobot/so101/sts3215_03a_v1.stl" />
-			</geometry>
-			<material name="sts3215" />
-		</visual>
-		<collision>
-			<origin xyz="-0.1224 0.0052 0.0187" rpy="-3.14159 -3.58047e-15 -3.14159" />
-			<geometry>
-				<mesh filename="package://robot_description/meshes/lerobot/so101/sts3215_03a_v1.stl" />
-			</geometry>
-		</collision>
-	</link>
-	<!-- Link wrist -->
-	<link name="wrist">
-		<inertial>
-			<origin xyz="-0.000103312 -0.0386143 0.0281156" rpy="0 0 0" />
-			<mass value="0.079" />
-			<inertia ixx="3.68263e-05" ixy="1.7893e-08" ixz="-5.28128e-08" iyy="2.5391e-05"
-				iyz="3.6412e-06" izz="2.1e-05" />
-		</inertial>
-		<!-- Part sts3215_03a_no_horn_v1 -->
-		<visual>
-			<origin xyz="5.55112e-17 -0.0424 0.0306" rpy="1.5708 1.5708 0" />
-			<geometry>
-				<mesh
-					filename="package://robot_description/meshes/lerobot/so101/sts3215_03a_no_horn_v1.stl" />
-			</geometry>
-			<material name="sts3215" />
-		</visual>
-		<collision>
-			<origin xyz="5.55112e-17 -0.0424 0.0306" rpy="1.5708 1.5708 0" />
-			<geometry>
-				<mesh
-					filename="package://robot_description/meshes/lerobot/so101/sts3215_03a_no_horn_v1.stl" />
-			</geometry>
-		</collision>
-		<!-- Part wrist_roll_pitch_so101_v2 -->
-		<visual>
-			<origin xyz="0 -0.028 0.0181" rpy="-1.5708 -1.5708 0" />
-			<geometry>
-				<mesh
-					filename="package://robot_description/meshes/lerobot/so101/wrist_roll_pitch_so101_v2.stl" />
-			</geometry>
-			<material name="3d_printed" />
-		</visual>
-		<collision>
-			<origin xyz="0 -0.028 0.0181" rpy="-1.5708 -1.5708 0" />
-			<geometry>
-				<mesh
-					filename="package://robot_description/meshes/lerobot/so101/wrist_roll_pitch_so101_v2.stl" />
-			</geometry>
-		</collision>
-	</link>
-	<!-- Link gripper -->
-	<link name="gripper">
-		<inertial>
-			<origin xyz="0.000213627 0.000245138 -0.025187" rpy="0 0 0" />
-			<mass value="0.087" />
-			<inertia ixx="2.75087e-05" ixy="-3.35241e-07" ixz="-5.7352e-06" iyy="4.33657e-05"
-				iyz="-5.17847e-08" izz="3.45059e-05" />
-		</inertial>
-		<!-- Part sts3215_03a_v1_5 -->
-		<visual>
-			<origin xyz="0.0077 0.0001 -0.0234" rpy="-1.5708 -5.55112e-17 -1.38213e-14" />
-			<geometry>
-				<mesh filename="package://robot_description/meshes/lerobot/so101/sts3215_03a_v1.stl" />
-			</geometry>
-			<material name="sts3215" />
-		</visual>
-		<collision>
-			<origin xyz="0.0077 0.0001 -0.0234" rpy="-1.5708 -5.55112e-17 -1.38213e-14" />
-			<geometry>
-				<mesh filename="package://robot_description/meshes/lerobot/so101/sts3215_03a_v1.stl" />
-			</geometry>
-		</collision>
-		<!-- Part wrist_roll_follower_so101_v1 -->
-		<visual>
-			<origin xyz="5.55112e-17 -0.000218214 0.000949706"
-				rpy="-3.14159 -5.55112e-17 -9.17912e-24" />
-			<geometry>
-				<mesh
-					filename="package://robot_description/meshes/lerobot/so101/wrist_roll_follower_so101_v1.stl" />
-			</geometry>
-			<material name="3d_printed" />
-		</visual>
-		<collision>
-			<origin xyz="5.55112e-17 -0.000218214 0.000949706"
-				rpy="-3.14159 -5.55112e-17 -9.17912e-24" />
-			<geometry>
-				<mesh
-					filename="package://robot_description/meshes/lerobot/so101/wrist_roll_follower_so101_v1.stl" />
-			</geometry>
-		</collision>
-	</link>
-	<!-- Link jaw -->
-	<link name="jaw">
-		<inertial>
-			<origin xyz="-0.00157495 -0.0300244 0.0192755" rpy="0 0 0" />
-			<mass value="0.012" />
-			<inertia ixx="6.61427e-06" ixy="-3.19807e-07" ixz="-5.90717e-09" iyy="1.89032e-06"
-				iyz="-1.09945e-07" izz="5.28738e-06" />
-		</inertial>
-		<!-- Part moving_jaw_so101_v1 -->
-		<visual>
-			<origin xyz="-5.55112e-17 -1.94746e-17 0.0189" rpy="9.53145e-17 -4.66093e-24 0" />
-			<geometry>
-				<mesh filename="package://robot_description/meshes/lerobot/so101/moving_jaw_so101_v1.stl" />
-			</geometry>
-			<material name="3d_printed" />
-		</visual>
-		<collision>
-			<origin xyz="-5.55112e-17 -1.94746e-17 0.0189" rpy="9.53145e-17 -4.66093e-24 0" />
-			<geometry>
-				<mesh filename="package://robot_description/meshes/lerobot/so101/moving_jaw_so101_v1.stl" />
-			</geometry>
-		</collision>
-	</link>
-	<!-- Link tcp (virtual Tool Center Point) -->
-	<!--
-	  Pure translation along gripper -Z (finger extension line); orientation
-	  identical to the gripper link (no relative rotation). Carries only a tiny
-	  visual marker (a small sphere) for RViz debugging, no collision geometry,
-	  so it never affects planning or collision checking.
-	-->
-	<material name="tcp_marker">
-		<color rgba="0.1 0.9 0.2 0.9" />
-	</material>
-	<link name="tcp">
-		<visual>
-			<origin xyz="0 0 0" rpy="0 0 0" />
-			<geometry>
-				<sphere radius="0.008" />
-			</geometry>
-			<material name="tcp_marker" />
-		</visual>
-	</link>
-	<joint name="gripper_to_tcp" type="fixed">
-		<origin xyz="$(arg tcp_offset_x) 0 $(arg tcp_offset_z)" rpy="0 0 0" />
-		<parent link="gripper" />
-		<child link="tcp" />
-	</joint>
-	<!-- Joint from gripper to jaw -->
-	<joint name="6" type="revolute">
-		<origin xyz="0.0202 0.0188 -0.0234" rpy="1.5708 0.209440 0.000001" />
-		<parent link="gripper" />
-		<child link="jaw" />
-		<axis xyz="0 0 1" />
-		<!-- Gripper joint: 0.0 = closed, 1.0 = open (similar to SO-ARM100) -->
-		<limit effort="10" velocity="10" lower="0.0" upper="1.0"/>
-	</joint>
-	<transmission name="6_trans">
-		<type>transmission_interface/SimpleTransmission</type>
-		<joint name="6">
-			<hardwareInterface>hardware_interface/PositionJointInterface</hardwareInterface>
-		</joint>
-		<actuator name="motor6">
-			<hardwareInterface>hardware_interface/PositionJointInterface</hardwareInterface>
-			<mechanicalReduction>1</mechanicalReduction>
-		</actuator>
-	</transmission>
-	<!-- Joint from wrist to gripper -->
-	<joint name="5" type="revolute">
-		<origin xyz="0 -0.0611 0.0181" rpy="1.5708 -9.38083e-08 3.14159" />
-		<parent link="wrist" />
-		<child link="gripper" />
-		<axis xyz="0 0 1" />
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
File: src/robot_description/urdf/lerobot/so101/so101_cameras.xacro (robot description, xacro)
@@ -1,77 +1,5 @@
 <?xml version="1.0"?>
 <robot xmlns:xacro="http://www.ros.org/wiki/xacro">
-    <!-- ============================================= -->
-    <!-- Wrist Camera (mounted on gripper body)      -->
-    <!-- ============================================= -->
-    <link name="wrist_camera_link">
-        <inertial>
-            <origin xyz="0 0 0" rpy="0 0 0"/>
-            <mass value="0.01"/>
-            <inertia ixx="0.001" ixy="0" ixz="0" iyy="0.001" iyz="0" izz="0.001"/>
-        </inertial>
-    </link>
-    <joint name="wrist_camera_joint" type="fixed">
-        <parent link="gripper"/>
-        <child link="wrist_camera_link"/>
-        <!-- Camera at center of palm back-plate, aimed at jaw closing center -->
-        <origin xyz="0.002 0.061 -0.025" rpy="-3.14159 -0.4 -1.5708"/>
-    </joint>
-    <!-- Wrist Camera Sensor for Gazebo -->
-    <gazebo reference="wrist_camera_link">
-        <sensor type="camera" name="wrist_camera">
-            <update_rate>30</update_rate>
-            <camera>
-                <horizontal_fov>1.5708</horizontal_fov>  <!-- 90 degrees -->
-                <image>
-                    <width>640</width>
-                    <height>480</height>
-                    <format>R8G8B8</format>
-                </image>
-                <clip>
-                    <near>0.01</near>
-                    <far>100</far>
-                </clip>
-            </camera>
-            <always_on>true</always_on>
-            <visualize>true</visualize>
-            <topic>wrist_camera/image</topic>
-        </sensor>
-    </gazebo>
-    <!-- ============================================= -->
-    <!-- Top Camera (mounted above workspace)         -->
-    <!-- ============================================= -->
-    <link name="top_camera_link">
-        <inertial>
-            <origin xyz="0 0 0" rpy="0 0 0"/>
-            <mass value="0.01"/>
-            <inertia ixx="0.001" ixy="0" ixz="0" iyy="0.001" iyz="0" izz="0.001"/>
-        </inertial>
-    </link>
-    <joint name="top_camera_joint" type="fixed">
-        <parent link="world"/>
-        <child link="top_camera_link"/>
-        <!-- Position camera above the workspace, pointing down -->
-        <origin xyz="0.3 0.0 0.8" rpy="0 0 3.14159"/>
-    </joint>
-    <!-- Top Camera Sensor for Gazebo -->
-    <gazebo reference="top_camera_link">
-        <sensor type="camera" name="top_camera">
-            <update_rate>30</update_rate>
-            <camera>
-                <horizontal_fov>1.047</horizontal_fov>  <!-- 60 degrees -->
-                <image>
-                    <width>640</width>
-                    <height>480</height>
-                    <format>R8G8B8</format>
-                </image>
-                <clip>
-                    <near>0.1</near>
-                    <far>100</far>
-                </clip>
-            </camera>
-            <always_on>true</always_on>
-            <visualize>true</visualize>
-            <topic>top_camera/image</topic>
-        </sensor>
-    </gazebo>
+	<!-- SSOT wrapper: included content lives in so101_description. -->
+	<xacro:include filename="$(find so101_description)/urdf/lerobot/so101/so101_cameras.xacro" />
 </robot>
