Commit message: runtime: add robot runtime contract and so101 runtime unit
Introduce robot_runtime (capability vocabulary, facade, mock, conformance,
public interface description with model metadata) and ibrobot_msgs runtime
and motion services. Add feetech_sdk and so101 sdk/hardware/description/
motion/suite packages under src/robots/, relocate so101_hardware, add the
two-direction independence gate with a fixed runtime allow-list.

- Harden SO101SystemHardware bus access with bounded retries and
  consecutive-failure counting; fail the controller chain only after
  sustained read or write failures with the Feetech fault code logged.
- Spawn the read-only leader input source from the runtime profile
  (teleoperation.leader_source) with scattered declared parameters;
  serial and calibration stay runtime-owned.
- Derive public gripper limits from calibration authority on physical
  hardware and model the arm joints with the single-turn mechanical
  envelope.
- Point the OpenHarmony cross-build and release path lists, ruff
  first-party names, the core-gate exclusion list and the repository
  layout docs at src/robots/so101 and robot_runtime.

- Harden the runtime stop path: epoch fencing keeps a concurrent mode
  switch from reviving motion or clearing a fresh stop latch, cancel
  results are validated for the active mode's trajectory endpoints, and
  stop success requires the command controllers to be deactivated.
- Harden the Feetech bus: shared config validation before EPROM writes,
  registry updates on reconfiguration, duplicate/oversized sync-read
  rejection, subset-sized sync-read sessions, sign-magnitude speed
  clamping, rollback outcome surfacing, EAGAIN-safe serial writes,
  wheel-mode calibration skip, ping-based activation diagnostics, and a
  time-budgeted retry window derived from update_rate.
- Make the core independence gate honest: launch output goes to a log
  file, motion waits are bounded, and StopRuntime(HOLD) is actually
  called with latch, lifecycle and mode asserted; pin the LeKiwi
  FTServo fetch to the feetech_sdk revision.
- Fail closed before the first runtime status in the motion server with
  a parameterized freshness deadline; honor ROS_HOME and the calibrator
  key set when loading ISP overrides.

Co-Authored-By: gpt-6-astra
Co-Authored-By: glm-5.3
Co-Authored-By: claude-opus-5
Signed-off-by: XiaoqiangWu <wuxiaoqiang.rtos@huawei.com>

File: src/robot_description/urdf/lerobot/so101/so101_dual.urdf.xacro (robot description, xacro)
@@ -1,84 +1,6 @@
 <?xml version="1.0"?>
 <robot xmlns:xacro="http://www.ros.org/wiki/xacro" name="so101_dual">
-  <xacro:arg name="use_sim" default="false"/>
-  <xacro:arg name="port_1" default=""/>
-  <xacro:arg name="calib_file_left" default=""/>
-  <xacro:arg name="port_2" default=""/>
-  <xacro:arg name="calib_file_right" default=""/>
-  <xacro:arg name="reset_positions" default="{}"/>
-  <link name="base_link"/>
-  <xacro:macro name="so101_arm" params="side mount_y port calib_file">
-    <link name="base_${side}"/>
-    <link name="shoulder_${side}"/>
-    <link name="upper_arm_${side}"/>
-    <link name="lower_arm_${side}"/>
-    <link name="wrist_${side}"/>
-    <link name="gripper_${side}"/>
-    <link name="jaw_${side}"/>
-    <joint name="base_mount_${side}" type="fixed">
-      <parent link="base_link"/>
-      <child link="base_${side}"/>
-      <origin xyz="0 ${mount_y} 0" rpy="0 0 0"/>
-    </joint>
-    <joint name="joint1_${side}" type="revolute">
-      <origin xyz="0.0207909 -0.0230745 0.0948817" rpy="-3.14159 6.03684e-16 1.5708"/>
-      <parent link="base_${side}"/>
-      <child link="shoulder_${side}"/>
-      <axis xyz="0 0 1"/>
-      <limit effort="10" velocity="10" lower="-2.0693" upper="2.0709"/>
-    </joint>
-    <joint name="joint2_${side}" type="revolute">
-      <origin xyz="-0.0303992 -0.0182778 -0.0542" rpy="-1.5708 -1.5708 0"/>
-      <parent link="shoulder_${side}"/>
-      <child link="upper_arm_${side}"/>
-      <axis xyz="0 0 1"/>
-      <limit effort="10" velocity="10" lower="-1.92" upper="1.92"/>
-    </joint>
-    <joint name="joint3_${side}" type="revolute">
-      <origin xyz="-0.11257 -0.028 2.46331e-16" rpy="-1.22818e-15 5.75928e-16 1.5708"/>
-      <parent link="upper_arm_${side}"/>
-      <child link="lower_arm_${side}"/>
-      <axis xyz="0 0 1"/>
-      <limit effort="10" velocity="10" lower="-1.6813" upper="1.6828"/>
-    </joint>
-    <joint name="joint4_${side}" type="revolute">
-      <origin xyz="-0.1349 0.0052 1.65232e-16" rpy="3.2474e-15 2.86219e-15 -1.5708"/>
-      <parent link="lower_arm_${side}"/>
-      <child link="wrist_${side}"/>
-      <axis xyz="0 0 1"/>
-      <limit effort="10" velocity="10" lower="-1.65806" upper="1.65806"/>
-    </joint>
-    <joint name="joint5_${side}" type="revolute">
-      <origin xyz="0 -0.0611 0.0181" rpy="1.5708 -9.38083e-08 3.14159"/>
-      <parent link="wrist_${side}"/>
-      <child link="gripper_${side}"/>
-      <axis xyz="0 0 1"/>
-      <limit effort="10" velocity="10" lower="-2.9115" upper="2.9115"/>
-    </joint>
-    <joint name="joint6_${side}" type="revolute">
-      <origin xyz="0.0202 0.0188 -0.0234" rpy="1.5708 -5.14108e-17 -1.38655e-14"/>
-      <parent link="gripper_${side}"/>
-      <child link="jaw_${side}"/>
-      <axis xyz="0 0 1"/>
-      <limit effort="10" velocity="10" lower="0.0" upper="1.0"/>
-    </joint>
-    <ros2_control name="${side}_so101_system" type="system">
-      <hardware>
-        <xacro:unless value="$(arg use_sim)">
-          <plugin>so101_hardware/SO101SystemHardware</plugin>
-          <param name="port">${port}</param>
-          <param name="calib_file">${calib_file}</param>
-          <param name="reset_positions">$(arg reset_positions)</param>
-        </xacro:unless>
-      </hardware>
-      <joint name="joint1_${side}"><command_interface name="position"/><state_interface name="position"/><state_interface name="velocity"/><param name="id">1</param></joint>
-      <joint name="joint2_${side}"><command_interface name="position"/><state_interface name="position"/><state_interface name="velocity"/><param name="id">2</param></joint>
-      <joint name="joint3_${side}"><command_interface name="position"/><state_interface name="position"/><state_interface name="velocity"/><param name="id">3</param></joint>
-      <joint name="joint4_${side}"><command_interface name="position"/><state_interface name="position"/><state_interface name="velocity"/><param name="id">4</param></joint>
-      <joint name="joint5_${side}"><command_interface name="position"/><state_interface name="position"/><state_interface name="velocity"/><param name="id">5</param></joint>
-      <joint name="joint6_${side}"><command_interface name="position"/><state_interface name="position"/><state_interface name="velocity"/><param name="id">6</param></joint>
-    </ros2_control>
-  </xacro:macro>
-  <xacro:so101_arm side="left" mount_y="0.18" port="$(arg port_1)" calib_file="$(arg calib_file_left)"/>
-  <xacro:so101_arm side="right" mount_y="-0.18" port="$(arg port_2)" calib_file="$(arg calib_file_right)"/>
+	<!-- SSOT wrapper: the model lives in so101_description; this copy only
+	     redirects legacy consumers so the two trees can never diverge. -->
+	<xacro:include filename="$(find so101_description)/urdf/lerobot/so101/so101_dual.urdf.xacro" />
 </robot>

File: src/robot_description/urdf/lerobot/so101/so101_gazebo.xacro (robot description, xacro)
@@ -1,32 +1,5 @@
 <?xml version="1.0"?>
 <robot xmlns:xacro="http://www.ros.org/wiki/xacro">
-    <!-- Absolute path set at launch (gz_ros2_control); fallback keeps install-time find. -->
-    <xacro:arg name="gz_ros2_control_parameters_file" default="$(find so101_hardware)/config/so101_controllers.yaml"/>
-    <!-- ROS 2 Control -->
-    <gazebo>
-        <plugin filename="gz_ros2_control-system" name="gz_ros2_control::GazeboSimROS2ControlPlugin">
-            <parameters>$(arg gz_ros2_control_parameters_file)</parameters>
-        </plugin>
-    </gazebo>
-    <!-- ============================================= -->
-    <!-- Gazebo material: uniform dark (sts3215 black) -->
-    <!-- ============================================= -->
-    <!-- Gazebo cannot color individual visuals within a link separately.
-         Uniform black matches the real robot's dominant visual appearance. -->
-    <xacro:macro name="gz_black" params="link_name">
-        <gazebo reference="${link_name}">
-            <visual><material>
-                <ambient>0.12 0.12 0.12 1</ambient>
-                <diffuse>0.12 0.12 0.12 1</diffuse>
-                <specular>0.15 0.15 0.15 1</specular>
-            </material></visual>
-        </gazebo>
-    </xacro:macro>
-    <xacro:gz_black link_name="base"/>
-    <xacro:gz_black link_name="shoulder"/>
-    <xacro:gz_black link_name="upper_arm"/>
-    <xacro:gz_black link_name="lower_arm"/>
-    <xacro:gz_black link_name="wrist"/>
-    <xacro:gz_black link_name="gripper"/>
-    <xacro:gz_black link_name="jaw"/>
+	<!-- SSOT wrapper: included content lives in so101_description. -->
+	<xacro:include filename="$(find so101_description)/urdf/lerobot/so101/so101_gazebo.xacro" />
 </robot>

File: src/robot_description/urdf/lerobot/so101/so101_ros2_control.xacro (robot description, xacro)
@@ -1,93 +1,5 @@
 <?xml version="1.0"?>
 <robot xmlns:xacro="http://www.ros.org/wiki/xacro">
-    <xacro:arg name="use_sim" default="true"/>
-    <xacro:arg name="port" default="/dev/ttyACM0"/>
-    <xacro:arg name="calib_file" default=""/>
-    <xacro:arg name="reset_positions" default=""/>
-    <!-- sim_plugin: hardware plugin for simulation. Default = Gazebo.
-         MuJoCo: description.py passes "mujoco_ros2_control/MujocoSystemInterface" when platform=mujoco. -->
-    <xacro:arg name="sim_plugin" default="gz_ros2_control/GazeboSimSystem"/>
-    <xacro:arg name="mujoco_model" default=""/>
-    <xacro:arg name="camera_publish_rate" default=""/>
-    <ros2_control name="RobotSystem" type="system">
-        <xacro:if value="$(arg use_sim)">
-            <hardware>
-                <plugin>$(arg sim_plugin)</plugin>
-                <xacro:if value="${'$(arg mujoco_model)' != ''}">
-                    <param name="mujoco_model">$(arg mujoco_model)</param>
-                </xacro:if>
-                <xacro:if value="${'$(arg camera_publish_rate)' != ''}">
-                    <param name="camera_publish_rate">$(arg camera_publish_rate)</param>
-                </xacro:if>
-            </hardware>
-        </xacro:if>
-        <xacro:unless value="$(arg use_sim)">
-            <hardware>
-                <plugin>so101_hardware/SO101SystemHardware</plugin>
-                <param name="port">$(arg port)</param>
-                <param name="calib_file">$(arg calib_file)</param>
-                <param name="reset_positions">$(arg reset_positions)</param>
-            </hardware>
-        </xacro:unless>
-        <joint name="1">
-            <command_interface name="position">
-                <param name="min">-2.0693</param>
-                <param name="max">2.0709</param>
-                <param name="initial_value">0.0</param>
-            </command_interface>
-            <state_interface name="position" />
-            <state_interface name="velocity" />
-            <param name="id">1</param>
-        </joint>
-        <joint name="2">
-            <command_interface name="position">
-                <param name="min">-1.92</param>
-                <param name="max">1.92</param>
-                <param name="initial_value">0.0</param>
-            </command_interface>
-            <state_interface name="position" />
-            <state_interface name="velocity" />
-            <param name="id">2</param>
-        </joint>
-        <joint name="3">
-            <command_interface name="position">
-                <param name="min">-1.6813</param>
-                <param name="max">1.6828</param>
-                <param name="initial_value">0.0</param>
-            </command_interface>
-            <state_interface name="position" />
-            <state_interface name="velocity" />
-            <param name="id">3</param>
-        </joint>
-        <joint name="4">
-            <command_interface name="position">
-                <param name="min">-1.65806</param>
-                <param name="max">1.65806</param>
-                <param name="initial_value">0.0</param>
-            </command_interface>
-            <state_interface name="position" />
-            <state_interface name="velocity" />
-            <param name="id">4</param>
-        </joint>
-        <joint name="5">
-            <command_interface name="position">
-                <param name="min">-2.9115</param>
-                <param name="max">2.9115</param>
-                <param name="initial_value">0.0</param>
-            </command_interface>
-            <state_interface name="position" />
-            <state_interface name="velocity" />
-            <param name="id">5</param>
-        </joint>
-        <joint name="6">
-            <command_interface name="position">
-                <param name="min">0.0</param>
-                <param name="max">1.0</param>
-                <param name="initial_value">0.0</param>
-            </command_interface>
-            <state_interface name="position" />
-            <state_interface name="velocity" />
-            <param name="id">6</param>
-        </joint>
-    </ros2_control>
+	<!-- SSOT wrapper: included content lives in so101_description. -->
+	<xacro:include filename="$(find so101_description)/urdf/lerobot/so101/so101_ros2_control.xacro" />
 </robot>
